Commit message: add custom bot

File: urdf/udacity_bot_four_wheel.xacro (robot description, xacro)
@@ -1,4 +1,4 @@
 <?xml version='1.0'?>
-<robot name="udacity_bot"
+<robot name="udacity_bot_four_wheel"
   xmlns:xacro="http://www.ros.org/wiki/xacro">
   <xacro:include filename="$(find udacity_bot)/urdf/udacity_bot.gazebo" />
@@ -12,5 +12,5 @@
     <pose>0 0 0.1 0 0 0</pose>
     <inertial>
-      <mass value="15.0"/>
+      <mass value="50.0"/>
       <origin xyz="0.0 0 0" rpy=" 0 0 0"/>
       <inertia ixx="0.1" ixy="0" ixz="0" iyy="0.1" iyz="0" izz="0.1" />
@@ -73,5 +73,5 @@
     </visual>
   </link>
-  <link name="left_wheel">
+  <link name="front_left_wheel">
     <inertial>
       <origin xyz="0.0 0.0 0.0" rpy="0.0 1.5707 1.5707" />
@@ -92,13 +92,14 @@
     </visual>
   </link>
-  <joint type="continuous" name="left_wheel_hinge">
-    <origin xyz="0.0 0.15 0.0" rpy="0 0 0"/>
-    <child link="left_wheel"/>
-    <parent link="chassis"/>
-    <axis xyz="0 1 0" rpy="0 0 0"/>
-    <limit effort="10000" velocity="1000"/>
-    <joint_properties damping="1.0" friction="1.0"/>
-  </joint>
-  <link name="right_wheel">
+  <joint type="continuous" name="front_left_wheel_hinge">
+    <origin xyz="0.15 0.15 0.0" rpy="0 0 0"/>
+    <child link="front_left_wheel"/>
+    <parent link="chassis"/>
+    <axis xyz="0 1 0" rpy="0 0 0"/>
+    <limit effort="10000" velocity="1000"/>
+    <!-- increased damping to reduce the osscilations when robot stops getting acceleration -->
+    <joint_properties damping="10.0" friction="1.0"/>
+  </joint>
+  <link name="front_right_wheel">
     <inertial>
       <origin xyz="0.0 0.0 0.0" rpy="0.0 1.5707 1.5707" />
@@ -119,11 +120,68 @@
     </visual>
   </link>
-  <joint type="continuous" name="right_wheel_hinge">
-    <origin xyz="0.0 -0.15 0.0" rpy="0 0 0"/>
-    <child link="right_wheel"/>
-    <parent link="chassis"/>
-    <axis xyz="0 1 0" rpy="0 0 0"/>
-    <limit effort="10000" velocity="1000"/>
-    <joint_properties damping="1.0" friction="1.0"/>
+  <joint type="continuous" name="front_right_wheel_hinge">
+    <origin xyz="0.15 -0.15 0.0" rpy="0 0 0"/>
+    <child link="front_right_wheel"/>
+    <parent link="chassis"/>
+    <axis xyz="0 1 0" rpy="0 0 0"/>
+    <limit effort="10000" velocity="1000"/>
+    <!-- increased damping to reduce the osscilations when robot stops getting acceleration -->
+    <joint_properties damping="10.0" friction="1.0"/>
+  </joint>
+  <link name="back_left_wheel">
+    <inertial>
+      <origin xyz="0.0 0.0 0.0" rpy="0.0 1.5707 1.5707" />
+      <mass value="5.0"/>
+      <inertia ixx="0.1" ixy="0" ixz="0" iyy="0.1" iyz="0" izz="0.1" />
+    </inertial>
+    <collision name='collision'>
+      <origin xyz="0.0 0.0 0.0" rpy=" 0 1.5707 1.5707"/>
+      <geometry>
+        <cylinder radius="0.1" length="0.05"/>
+      </geometry>
+    </collision>
+    <visual name="lef_wheel_visual">
+      <origin xyz="0.0 0.0 0.0" rpy="0 1.5707 1.5707" />
+      <geometry>
+        <cylinder radius="0.1" length="0.05"/>
+      </geometry>
+    </visual>
+  </link>
+  <joint type="continuous" name="back_left_wheel_hinge">
+    <origin xyz="-0.15 0.15 0.0" rpy="0 0 0"/>
+    <child link="back_left_wheel"/>
+    <parent link="chassis"/>
+    <axis xyz="0 1 0" rpy="0 0 0"/>
+    <limit effort="10000" velocity="1000"/>
+    <!-- increased damping to reduce the osscilations when robot stops getting acceleration -->
+    <joint_properties damping="10.0" friction="1.0"/>
+  </joint>
+  <link name="back_right_wheel">
+    <inertial>
+      <origin xyz="0.0 0.0 0.0" rpy="0.0 1.5707 1.5707" />
+      <mass value="5.0"/>
+      <inertia ixx="0.1" ixy="0" ixz="0" iyy="0.1" iyz="0" izz="0.1" />
+    </inertial>
+    <collision name='collision'>
+      <origin xyz="0.0 0.0 0.0" rpy=" 0 1.5707 1.5707"/>
+      <geometry>
+        <cylinder radius="0.1" length="0.05"/>
+      </geometry>
+    </collision>
+    <visual name="right_wheel_visual">
+      <origin xyz="0.0 0.0 0.0" rpy="0 1.5707 1.5707" />
+      <geometry>
+        <cylinder radius="0.1" length="0.05"/>
+      </geometry>
+    </visual>
+  </link>
+  <joint type="continuous" name="back_right_wheel_hinge">
+    <origin xyz="-0.15 -0.15 0.0" rpy="0 0 0"/>
+    <child link="back_right_wheel"/>
+    <parent link="chassis"/>
+    <axis xyz="0 1 0" rpy="0 0 0"/>
+    <limit effort="10000" velocity="1000"/>
+    <!-- increased damping to reduce the osscilations when robot stops getting acceleration -->
+    <joint_properties damping="10.0" friction="1.0"/>
   </joint>
 <!--Camera-->
@@ -154,22 +212,22 @@
   </joint>
 <!--LIDAR-->
-<link name="hokuyo">
-    <origin>0. 0 0 0 0 0</origin>
-    <inertial>
-      <origin xyz="0 0 0" rpy="0 0 0"/>
-      <mass value ="0.1"/>
-      <inertia ixx="1e-6" ixy="0" ixz="0" iyy="1e-6" iyz="0" izz="1e-6"/>
-    </inertial>
-    <collision name="collision">
-      <origin xyz="0 0 0" rpy="0 0 0"/>
-      <geometry>
-        <box size="0.1 0.1 0.1" />
-      </geometry>
-    </collision>
-    <visual>
-      <geometry>
-        <mesh filename="package://udacity_bot/meshes/hokuyo.dae" />
-      </geometry>
-    </visual>
+  <link name="hokuyo">
+      <origin>0. 0 0 0 0 0</origin>
+      <inertial>
+        <origin xyz="0 0 0" rpy="0 0 0"/>
+        <mass value ="0.1"/>
+        <inertia ixx="1e-6" ixy="0" ixz="0" iyy="1e-6" iyz="0" izz="1e-6"/>
+      </inertial>
+      <collision name="collision">
+        <origin xyz="0 0 0" rpy="0 0 0"/>
+        <geometry>
+          <box size="0.1 0.1 0.1" />
+        </geometry>
+      </collision>
+      <visual>
+        <geometry>
+          <mesh filename="package://udacity_bot/meshes/hokuyo.dae" />
+        </geometry>
+      </visual>
   </link>
   <joint type="fixed" name="hokuyo_joint">
